File: btaudio/btaudio.kicad_sch (KiCad schematic)
At the start: 1 part, among them U1 EWM104-BT5125

Commit message: symbol
Changed lines of the file:
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@@
 	(symbol
 		(lib_id "EWM104-BT5125:EWM104-BT5125")
-		(at 128.27 99.06 0)
+		(at 127 81.28 0)
 		(unit 1)
 		(body_style 1)
@@
 		(fields_autoplaced yes)
 		(property "Reference" "U1"
-			(at 128.27 44.45 0)
+			(at 127 26.67 0)
 			(show_name no)
 			(do_not_autoplace no)
@@
 		)
 		(property "Value" "EWM104-BT5125"
-			(at 128.27 46.99 0)
+			(at 127 29.21 0)
 			(show_name no)
 			(do_not_autoplace no)
@@
 		)
 		(property "Footprint" "EWM104-BT5125:EWM104-BT5125"
-			(at 128.27 99.06 0)
+			(at 127 81.28 0)
 			(hide yes)
 			(show_name no)
@@
 		)
 		(property "Datasheet" "https://www.cdebyte.com/products/EWM104-BT5125(I2S)/2"
-			(at 128.27 99.06 0)
+			(at 127 81.28 0)
 			(hide yes)
 			(show_name no)
@@
 		)
 		(property "Description" "QCC5125 BLE5.1 Bluetooth Audio Module (DAC/I2S/SPDIF), 54-pad castellated"
-			(at 128.27 99.06 0)
+			(at 127 81.28 0)
 			(hide yes)
 			(show_name no)
@@
 			)
 		)
-		(pin "19"
+		(pin "27"
+		)
+		(pin "22"
+		)
+		(pin "10"
+		)
+		(pin "46"
+		)
+		(pin "45"
+		)
+		(pin "39"
+		)
+		(pin "5"
+		)
+		(pin "43"
 		)
 		(pin "21"
 		)
-		(pin "1"
+		(pin "33"
+		)
+		(pin "32"
+		)
+		(pin "48"
+		)
+		(pin "3"
+		)
+		(pin "25"
+		)
+		(pin "51"
+		)
+		(pin "30"
+		)
+		(pin "49"
+		)
+		(pin "34"
+		)
+		(pin "29"
+		)
+		(pin "18"
+		)
+		(pin "44"
+		)
+		(pin "11"
+		)
+		(pin "17"
+		)
+		(pin "23"
+		)
+		(pin "13"
+		)
+		(pin "52"
+		)
+		(pin "16"
+		)
+		(pin "31"
+		)
+		(pin "47"
+		)
+		(pin "50"
 		)
 		(pin "12"
 		)
-		(pin "15"
+		(pin "53"
+		)
+		(pin "54"
+		)
+		(pin "19"
+		)
+		(pin "7"
+		)
+		(pin "41"
+		)
+		(pin "8"
+		)
+		(pin "20"
+		)
+		(pin "1"
+		)
+		(pin "2"
+		)
+		(pin "9"
+		)
+		(pin "36"
 		)
 		(pin "26"
 		)
-		(pin "29"
+		(pin "37"
 		)
-		(pin "31"
+		(pin "35"
+		)
+		(pin "15"
+		)
+		(pin "42"
+		)
+		(pin "40"
+		)
+		(pin "38"
 		)
 		(pin "28"
 		)
-		(pin "13"
+		(pin "4"
 		)
-		(pin "7"
+		(pin "24"
 		)
-		(pin "2"
-		)
-		(pin "3"
-		)
-		(pin "9"
-		)
-		(pin "5"
-		)
-		(pin "4"
+		(pin "14"
 		)
 		(pin "6"
 		)
-		(pin "8"
-		)
-		(pin "10"
-		)
-		(pin "11"
-		)
-		(pin "14"
-		)
-		(pin "16"
-		)
-		(pin "17"
-		)
-		(pin "18"
-		)
-		(pin "20"
-		)
-		(pin "22"
-		)
-		(pin "23"
-		)
-		(pin "24"
-		)
-		(pin "25"
-		)
-		(pin "27"
-		)
-		(pin "30"
-		)
-		(pin "34"
-		)
-		(pin "45"
-		)
-		(pin "52"
-		)
-		(pin "41"
-		)
-		(pin "51"
-		)
-		(pin "46"
-		)
-		(pin "32"
-		)
-		(pin "42"
-		)
-		(pin "50"
-		)
-		(pin "35"
-		)
-		(pin "54"
-		)
-		(pin "38"
-		)
-		(pin "43"
-		)
-		(pin "44"
-		)
-		(pin "48"
-		)
-		(pin "49"
-		)
-		(pin "39"
-		)
-		(pin "53"
-		)
-		(pin "36"
-		)
-		(pin "37"
-		)
-		(pin "33"
-		)
-		(pin "40"
-		)
-		(pin "47"
-		)
 		(instances

Commit message: some progress schema
Parts:
- added C1: 10uF, Capacitor_SMD:C_0805_2012Metric_Pad1.18x1.45mm_HandSolder, symbol Device:C
- added C10, C11, C12, C16, C17: 10uF, symbol Device:C
- added C13, C14, C15, C18, C19, C20, C4, C5, C7, C8, C9: 100nF, symbol Device:C
- added C2, C3: 4.7uF, Capacitor_SMD:C_0805_2012Metric_Pad1.18x1.45mm_HandSolder, symbol Device:C
- added C21, C22, C23: 1uF, symbol Device:C
- added C6: 4.7uF, symbol Device:C
- added D1: Blue, LED_SMD:LED_0805_2012Metric_Pad1.15x1.40mm_HandSolder, symbol Device:LED
- added D2: Green, LED_SMD:LED_0805_2012Metric_Pad1.15x1.40mm_HandSolder, symbol Device:LED
- added D3: Red, LED_SMD:LED_0805_2012Metric_Pad1.15x1.40mm_HandSolder, symbol Device:LED
- added IC1: MCP73871-2CCI_ML, MCP73871-2CCI_ML:QFN50P400X400X100-21N-D, symbol MCP73871-2CCI_ML:MCP73871-2CCI_ML
- added J1: Vbat, Connector_PinSocket_2.00mm:PinSocket_1x02_P2.00mm_Vertical, symbol Connector:Conn_01x02_Socket
- added J2: USB_C_Receptacle_USB2.0_16P, Connector_USB:USB_C_Receptacle_HRO_TYPE-C-31-M-12, symbol Connector:USB_C_Receptacle_USB2.0_16P
- added J3: Load, Connector_PinSocket_2.00mm:PinSocket_1x02_P2.00mm_Vertical, symbol Connector:Conn_01x02_Socket
- added JP3: Timer Jumper, Jumper:SolderJumper-2_P1.3mm_Bridged_RoundedPad1.0x1.5mm, symbol Jumper:Jumper_2_Bridged
- added J_HP: AudioJack_3.5mm, symbol AudioJack3
- added R1, R2: 5.1k, Resistor_SMD:R_0805_2012Metric_Pad1.20x1.40mm_HandSolder, symbol Device:R
- added R3: 330k, Resistor_SMD:R_0805_2012Metric_Pad1.20x1.40mm_HandSolder, symbol Device:R
- added R4: 110k, Resistor_SMD:R_0805_2012Metric_Pad1.20x1.40mm_HandSolder, symbol Device:R
- added R5: 1k, Resistor_SMD:R_0805_2012Metric_Pad1.20x1.40mm_HandSolder, symbol Device:R
- added R50: 100kΩ, Resistor_SMD:R_0805_2012Metric_Pad1.20x1.40mm_HandSolder, symbol Device:R
- added R6, R7, R8: 470, Resistor_SMD:R_0805_2012Metric_Pad1.20x1.40mm_HandSolder, symbol Device:R
- added R9: 25k, Resistor_SMD:R_0805_2012Metric_Pad1.20x1.40mm_HandSolder, symbol Device:R
- added TH1: NTC B3950 10k, Connector_PinSocket_2.00mm:PinSocket_1x02_P2.00mm_Vertical, symbol Device:Thermistor_NTC
- added U2: PCM5102AQPWRQ1, SOP65P640X120-20N, symbol PCM5102AQPWRQ1:PCM5102AQPWRQ1
- added U3: TPA6132A2RTET, QFN50P300X300X80-17N-D, symbol TPA6132A2RTET:TPA6132A2RTET
- added U5: MCP1700x-330xxTT, Package_TO_SOT_SMD:SOT-23, symbol Regulator_Linear:MCP1700x-330xxTT
Connections:
- net VIN: now reaches U1.10 (VCHG)
- net VIN: now also C7.1
- net VBAT: now reaches U1.14 (VBAT)
- net VBAT: now also C11.1, C8.1, R50.1
- net GND: now reaches U1.15 (GND)
- net GND: now also U1.21 (GND), U1.38 (GND), U1.44 (GND), U1.45 (GND), U1.47 (GND), C1.2, C10.2, C11.2, C12.2, C13.2, C14.2, C15.2, C16.2, C17.2, C18.2, C19.2, C2.2, C20.2, C3.2, C4.2, C5.2, C6.2, C7.2, C8.2, C9.2, IC1.10 (VSS_1), IC1.11 (VSS_2), IC1.21 (EP), IC1.4 (PROG2), J1.2 (Pin_2), J2.A1 (GND), J2.A12 (GND), J2.B1 (GND), J2.B12 (GND), J2.S1 (SHIELD), J3.2 (Pin_2), JP3.2 (B), J_HP.3 (S), R1.2, R2.2, R4.2, R5.2, R9.2, TH1.2, U2.10 (DEMP), U2.11 (FLT), U2.16 (FMT), U2.19 (DGND), U2.3 (CPGND), U2.9 (AGND), U3.1 (INL-), U3.10 (PGND), U3.15 (SGND), U3.17 (EP), U3.4 (INR-), U3.8 (HPVSS), U5.1 (GND)
- net +3V3: now reaches U1.23 (VDD_PADS1)
- net +3V3: now also U1.24 (VDD_PADS3_7), C10.1, C13.1, C14.1, C15.1, C16.1, C17.1, C18.1, C20.1, C5.1, C6.1, C9.1, U2.1 (CPVDD), U2.17 (XSMT), U2.20 (DVDD), U2.8 (AVDD), U3.12 (HPVDD), U3.13 (EN), U5.2 (VO)
- net I2S_SDATA: now reaches U1.3 (I2S_SDATA/SPDIF_OUT)
- net I2S_SDATA: now also U2.14 (DIN)
- net I2S_LRCK: now reaches U1.4 (I2S_LRCK)
- net I2S_LRCK: now also U2.15 (LRCK)
- net I2S_SCK: now reaches U1.5 (I2S_SCK)
- net I2S_SCK: now also U2.13 (BCK)
- net I2S_MCLK: now reaches U1.6 (I2S_MCLK)
- net I2S_MCLK: now also U2.12 (SCK)
- new net: IC1.5 (THERM), TH1.1
- new net: IC1.6 (~{PG}), R6.2
- new net: IC1.7 (STAT2), R7.2
- new net: IC1.8 (STAT1/~{LBO}), R8.2
- new net: D2.1 (K), R7.1
- new net: C23.1, U3.11 (CPP)
- new net: C23.2, U3.9 (CPN)
- new net: J2.B5 (CC2), R2.1
- new net: D1.1 (K), R6.1
- new net: J2.A5 (CC1), R1.1
- new net: C22.2, U3.3 (INR+)
- new net: C21.2, U3.2 (INL+)
- new net: D3.1 (K), R8.1
- new net D+: J2.A6 (D+), J2.B6 (D+)
- new net D-: J2.A7 (D-), J2.B7 (D-)
- new net GAIN0: U3.6 (G0)
- new net GAIN1: U3.7 (G1)
- new net HP_OUTL: J_HP.1 (T), U3.16 (OUTL)
- new net HP_OUTR: J_HP.2 (R), U3.5 (OUTR)
- new net LDOO: C19.1, U2.18 (LDOO)
- new net Load: C2.1, IC1.1 (OUT_1), IC1.20 (OUT_2), J3.1 (Pin_1)
- new net PCM_OUTL: C21.1, U2.6 (OUTL)
- new net PCM_OUTR: C22.1, U2.7 (OUTR)
- new net PROG1: IC1.13 (PROG1), R5.1
- new net PROG3: IC1.12 (PROG3), R9.1
- new net SEL: C1.1, D1.2 (A), D2.2 (A), D3.2 (A), IC1.17 (CE), IC1.18 (IN_1), IC1.19 (IN_2), IC1.3 (SEL), J2.A4 (VBUS), J2.A9 (VBUS), J2.B4 (VBUS), J2.B9 (VBUS), R3.1
- new net SYS_RC: C12.1, R50.2
- new net TE: IC1.9 (~{TE}), JP3.1 (A)
- new net VPCC: IC1.2 (VPCC), R3.2, R4.1
- new net Vbat: C3.1, C4.1, IC1.14 (VBAT_1), IC1.15 (VBAT_2), IC1.16 (VBAT_SENSE), J1.1 (Pin_1), U5.3 (VI)
- no-connect marks 0 -> 38
Other:
- note added: "(low for USB port, high for AC-DC adapter)"
- note added: "1.23V = (110k / (R1 + 110k)) * 5V"
- note added: "100mA"
- note added: "500mA"
- note added: "AC/DC Adapter or USB Port"
- note added: "Decoupling: 100nF X5R 0402 + 10uF X5R 0805"
- note added: "Device Charge Enable"
- note added: "Enabled when CE = high"
- note added: "Enables Safety Timer when active-low"
- note added: "Fast charge current regulation setting with SEL = high. Preconditioning set point for both USB port and AC-DC adapter"
- note added: "I = 1000V / Rprog1"
- note added: "I = 1000V / Rprog3"
- note added: "If Source can't supply enough current, causing Vin to drop, VPCC will lower the drawn current to sustain 5V at Vin."
- note added: "Input type selection"
- note added: "MCP1700: VBAT -> 3V3"
- note added: "MCP73871"
- note added: "NOTE: AC coupling caps 1uF between U2 OUTL/OUTR and U3 INL+/INR+"
- note added: "NOTE: ANT (U1 pin46): Johanson 0433AT62A0020E + pi-match network (see PLAN.md)"
- note added: "NOTE: Add 2N7002 MOSFET: G=SYS_RC, D=SYS_CTRL pin13, S=GND"
- note added: "PROG1: Charge Current Regulation Set"
- note added: "PROG2: USB-Port Current Regulation Set"
- note added: "PROG3: Charge Termination"
- note added: "R1"
- note added: "R1 = 337k"
- note added: "R2"
- note added: "Rprog1 = 1k -> 1.0A"
- note added: "Rprog1 = 2k -> 0.5A"
- note added: "Rprog1 = 5k -> 0.2A"
- note added: "Rprog3 = 25k -> 40mA"
- note added: "Stand-Alone System Load Sharing and Li-Ion/Li-Polymer Battery Charge Management Controller"
- note added: "Termination set point for both AC-DC adapter and USB port"
- note added: "Timer Enable"
- note added: "USB port input current limit selection when SEL = Low (Low = 100 mA, High = 500 mA)"
- note added: "Voltage Proportional Charge Control"
- note added: "Vvpcc = (R2 / (R1 + R2)) * Vin = 1.23V"

Commit message: PCM5102A Schema done
Parts:
- added C24, C26: 100nF, symbol Device:C
- added C25, C27, C30, C31: 10uF, symbol Device:C_Polarized
- added C28, C29: 2.2nF, symbol Device:C
- added R10, R11: 470, symbol Device:R
- C15: value 100nF -> 2.2uF
- C16: value 10uF -> 2.2uF
- renumbered J_HP to J_HP1
Connections:
- net +3V3: now also C24.1, C25.1, C30.1, C31.1; no longer C15.1, C16.1
- net GND: now also C16.1, U2.12 (SCK), C24.2, C25.2, C26.2, C27.2, C28.2, C29.2, C30.2, C31.2; no longer C15.2, C16.2
- net LDOO: no longer U2.18 (LDOO)
- net PCM_OUTL: now also R10.1
- net PCM_OUTR: now also R11.1
- net CAPP: now reaches U2.2 (CAPP)
- net CAPP: now also C15.1
- net CAPM: now reaches U2.4 (CAPM)
- net CAPM: now also C15.2
- net VNEG: now reaches U2.5 (VNEG)
- net VNEG: now also C16.2
- net I2S_MCLK: no longer names the net of U1.6 (I2S_MCLK)
- net I2S_MCLK: no longer U2.12 (SCK)
- new net: C26.1, C27.1, U2.18 (LDOO)
- new net LP_OUTL: C28.1, R10.2
- new net LP_OUTR: C29.1, R11.2
- no-connect marks 38 -> 36
Other:
- note added: "Disable De-Emphasis"
- note added: "Disable Mute"
- note added: "Enable Interal PLL"
- note added: "Internal 1.8V"
- note added: "LAYOUT KONZEPT: PARTITIONING Jeder GND-Pin bekommt direkt daneben ein eigenes Via Seperation der Analog und Digital Ströme durch platzierung"
- note added: "Left/Right Clock"
- note added: "PCM Output Low Pass"
- note added: "PCM5102A: I2S -> Line Out L/R"
- note added: "Set "Normal Latency""
- moved on the sheet: C13, U2

Commit message: TPA6132A schema done
Parts:
- removed C17: 10uF, symbol Device:C
- removed C18, C19, C20: 100nF, symbol Device:C
- added C32, C34: 2.2uF, symbol Device:C
- added C33: 1uF, symbol Device:C
- added JP1: GAIN0, symbol Jumper:SolderJumper_3_Open
- added JP2: GAIN1, symbol Jumper:SolderJumper_3_Open
- added R12: 10k, symbol Device:R
Connections:
- net +3V3: now also U3.14 (VDD), C34.1, JP1.1 (A), JP2.1 (A); no longer U3.12 (HPVDD), U3.13 (EN)
- net GAIN0: now also JP1.2 (C)
- net GAIN1: now also JP2.2 (C)
- net GND: now also U3.2 (INL+), U3.3 (INR+), C32.2, C33.2, C34.2, JP1.3 (B), JP2.3 (B), R12.2; no longer U3.1 (INL-), U3.4 (INR-), U3.8 (HPVSS)
- net LP_OUTL: now also C21.1
- net LP_OUTR: now also C22.1
- net PCM_OUTL: no longer C21.1
- net PCM_OUTR: no longer C22.1
- net VBAT: now also U1.7 (VBAT_SENSE)
- net VIN: now also U1.11 (VCHG_SENSE)
- net at C22.2: now also U3.4 (INR-); no longer U3.3 (INR+)
- net at C21.2: now also U3.1 (INL-); no longer U3.2 (INL+)
- net AMP_EN: now reaches U1.54 (PIO[20](AMP_EN))
- net AMP_EN: now also U3.13 (EN), R12.1
- new net: C32.1, U3.12 (HPVDD)
- new net: C33.1, U3.8 (HPVSS)
- no-connect marks 36 -> 35
Other:
- note added: "Headphone Amplifier: PCM -> AUX"
- note added: "LAYOUT KONZEPT: SGND muss direkt bei der AUX-Buchse aufs GND Plane"
- note added: "X5R/X7R"
- note removed: "NOTE: AC coupling caps 1uF between U2 OUTL/OUTR and U3 INL+/INR+"
- moved on the sheet: C23, J_HP1, R50, U3

Commit message: schema done
Parts:
- removed C1: 10uF, Capacitor_SMD:C_0805_2012Metric_Pad1.18x1.45mm_HandSolder, symbol Device:C
- removed C10, C12: 10uF, symbol Device:C
- removed C2, C3: 4.7uF, Capacitor_SMD:C_0805_2012Metric_Pad1.18x1.45mm_HandSolder, symbol Device:C
- removed C6: 4.7uF, symbol Device:C
- removed C9: 100nF, symbol Device:C
- removed D1: Blue, LED_SMD:LED_0805_2012Metric_Pad1.15x1.40mm_HandSolder, symbol Device:LED
- removed D2: Green, LED_SMD:LED_0805_2012Metric_Pad1.15x1.40mm_HandSolder, symbol Device:LED
- removed D3: Red, LED_SMD:LED_0805_2012Metric_Pad1.15x1.40mm_HandSolder, symbol Device:LED
- removed IC1: MCP73871-2CCI_ML, MCP73871-2CCI_ML:QFN50P400X400X100-21N-D, symbol MCP73871-2CCI_ML:MCP73871-2CCI_ML
- removed J3: Load, Connector_PinSocket_2.00mm:PinSocket_1x02_P2.00mm_Vertical, symbol Connector:Conn_01x02_Socket
- removed JP3: Timer Jumper, Jumper:SolderJumper-2_P1.3mm_Bridged_RoundedPad1.0x1.5mm, symbol Jumper:Jumper_2_Bridged
- removed R1, R2: 5.1k, Resistor_SMD:R_0805_2012Metric_Pad1.20x1.40mm_HandSolder, symbol Device:R
- removed R3: 330k, Resistor_SMD:R_0805_2012Metric_Pad1.20x1.40mm_HandSolder, symbol Device:R
- removed R50: 100kΩ, Resistor_SMD:R_0805_2012Metric_Pad1.20x1.40mm_HandSolder, symbol Device:R
- removed R6, R7, R8: 470, Resistor_SMD:R_0805_2012Metric_Pad1.20x1.40mm_HandSolder, symbol Device:R
- removed R9: 25k, Resistor_SMD:R_0805_2012Metric_Pad1.20x1.40mm_HandSolder, symbol Device:R
- removed TH1: NTC B3950 10k, Connector_PinSocket_2.00mm:PinSocket_1x02_P2.00mm_Vertical, symbol Device:Thermistor_NTC
- added AE1: Ceramic Antenna, symbol Device:Antenna
- added AE2: IPEX Plug, symbol Device:Antenna
- added C17, C18: NC, symbol Device:C
- added D4, D5: LED, LED_THT:LED_D5.0mm, symbol PCM_SL_Devices:LED
- added L1: 0 Ohm, symbol Device:L
- added NT1: NetTie, NetTie:NetTie-2_SMD_Pad0.5mm, symbol Device:NetTie_2
- added R14, R15: 1k, symbol Device:R
- added R16, R17: 0, symbol Device:R
- added SW1: POWER_SW, symbol Switch:SW_Push
- added SW2: PLAY/VOL+, symbol Switch:SW_Push
- added SW3: PAUSE/VOL-, symbol Switch:SW_Push
- added SW4: PREV/BT PAIRING, symbol Switch:SW_Push
- added SW5: NEXT/BT DISCONNECT, symbol Switch:SW_Push
- added SW6: SOFT RESET, symbol Switch:SW_Push
- C4, C5, C7: value 100nF -> 1uF
- J1: value Vbat -> BAT_CON; footprint Connector_PinSocket_2.00mm:PinSocket_1x02_P2.00mm_Vertical -> Connector_JST:JST_SH_SM02B-SRSS-TB_1x02-1MP_P1.00mm_Horizontal
- JP1: footprint (none) -> Jumper:SolderJumper-3_P1.3mm_Open_RoundedPad1.0x1.5mm
- R4: value 110k -> 5.1k; footprint Resistor_SMD:R_0805_2012Metric_Pad1.20x1.40mm_HandSolder -> (none)
- R5: value 1k -> 5.1k; footprint Resistor_SMD:R_0805_2012Metric_Pad1.20x1.40mm_HandSolder -> (none)
- U1: footprint EWM104-BT5125:EWM104-BT5125 -> EWM104-BT5125-PCB:EWM104-BT5125(KiCAD)
- U2: footprint SOP65P640X120-20N -> PCM5102AQPWRQ1:SOP65P640X120-20N
- U3: footprint QFN50P300X300X80-17N-D -> TPA6132A2RTET:QFN50P300X300X80-17N-D
Connections:
- net PROG1 is gone; now on an unnamed net: R5.1
- net SEL is gone; now on net VIN: J2.A4 (VBUS), J2.A9 (VBUS), J2.B4 (VBUS), J2.B9 (VBUS)
- net VPCC is gone; now on an unnamed net: R4.1
- net D+: now also U1.9 (USB_DP)
- net D-: now also U1.8 (USB_DN)
- net GND: now also J1.1 (Pin_1), J2.SH (SHIELD), C17.2, C18.2, NT1.1, SW2.1, SW3.1, SW4.1, SW5.1, SW6.1; no longer J1.2 (Pin_2), J2.S1 (SHIELD), J_HP1.3 (S), U3.15 (SGND)
- net VBAT: now also C4.1, U5.3 (VI), R14.2, R15.2, SW1.1
- net VIN: now also J1.2 (Pin_2)
- net at U1.13 (SYS_CTRL): now also SW1.2
- net at U1.16 (AIO[0]/LED[0]): now also D4.1
- net at U1.17 (AIO[1]/LED[1]): now also D5.1
- net at U1.25 (PIO[4]): now also SW4.2
- net at U1.26 (PIO[3]): now also SW3.2
- net at U1.28 (PIO[5]): now also SW5.2
- net at U1.31 (PIO[2]): now also SW2.2
- net at U1.32 (~{RST}/PIO[1]): now also SW6.2
- net at U1.46 (ANT): now also C17.1, L1.1
- removed net Vbat: C4.1, J1.1 (Pin_1), U5.3 (VI)
- new net: C18.1, L1.2, R16.2, R17.2
- new net: D5.2, R15.1
- new net: AE1.1 (A), R17.1
- new net: AE2.1 (A), R16.1
- new net: D4.2, R14.1
- new net SGND_TRACE: J_HP1.3 (S), NT1.2, U3.15 (SGND)
- no-connect marks 35 -> 27
Other:
- note added: "EWM104-BT5125(I2S) QCC5125"
- note added: "Spannungspegel für GPIO und I2S"
- note removed: "(low for USB port, high for AC-DC adapter)"
- note removed: "1.23V = (110k / (R1 + 110k)) * 5V"
- note removed: "100mA"
- note removed: "500mA"
- note removed: "AC/DC Adapter or USB Port"
- note removed: "Decoupling: 100nF X5R 0402 + 10uF X5R 0805"
- note removed: "Device Charge Enable"
- note removed: "Enabled when CE = high"
- note removed: "Enables Safety Timer when active-low"
- note removed: "Fast charge current regulation setting with SEL = high. Preconditioning set point for both USB port and AC-DC adapter"
- note removed: "I = 1000V / Rprog1"
- note removed: "I = 1000V / Rprog3"
- note removed: "If Source can't supply enough current, causing Vin to drop, VPCC will lower the drawn current to sustain 5V at Vin."
- note removed: "Input type selection"
- note removed: "MCP73871"
- note removed: "NOTE: ANT (U1 pin46): Johanson 0433AT62A0020E + pi-match network (see PLAN.md)"
- note removed: "NOTE: Add 2N7002 MOSFET: G=SYS_RC, D=SYS_CTRL pin13, S=GND"
- note removed: "PROG1: Charge Current Regulation Set"
- note removed: "PROG2: USB-Port Current Regulation Set"
- note removed: "PROG3: Charge Termination"
- note removed: "R1"
- note removed: "R1 = 337k"
- note removed: "R2"
- note removed: "Rprog1 = 1k -> 1.0A"
- note removed: "Rprog1 = 2k -> 0.5A"
- note removed: "Rprog1 = 5k -> 0.2A"
- note removed: "Rprog3 = 25k -> 40mA"
- note removed: "Stand-Alone System Load Sharing and Li-Ion/Li-Polymer Battery Charge Management Controller"
- note removed: "Termination set point for both AC-DC adapter and USB port"
- note removed: "Timer Enable"
- note removed: "USB port input current limit selection when SEL = Low (Low = 100 mA, High = 500 mA)"
- note removed: "Voltage Proportional Charge Control"
- note removed: "Vvpcc = (R2 / (R1 + R2)) * Vin = 1.23V"
- company: (none) -> EWM104-BT5125(I2S) - QCC5125
- title: (none) -> btaudio
- moved on the sheet: C11, C13, C14, C15, C16, C21, C22, C23, C24, C25, C26, C27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
