File: btaudio/btaudio.kicad_pcb (KiCad board)
At the start: 4 copper layers, 22 x 51 mm, 49 parts, among them J1 BTNS, J2 USB_C_Receptacle_USB2.0_16P, J3 Audio, J6 Battery, SW1 POWER_SW, SW6 SOFT RESET, U1 EWM104-BT5125, U2 PCM5102AQPWRQ1, U3 TPA6132A2RTET, U5 MCP1700x-330xxTT

Commit message: finished layout & aesthetics
Parts:
- added G***: LOGO, LOGO, B.Cu at (143.0, 92.4)
Routing:
- net /VBAT: track 48.6 -> 49.4 mm
- net GND: vias 72 -> 73
Other:
- board text added: "2"
- board text added: "3"
- board text added: "4"
- board text added: "AUDIO OUT"
- board text added: "BT->I2S->Amp EWM104-BT5125(I2S) QCC5125"
- board text added: "DH"
- board text added: "G1"
- board text added: "G2"
- board text added: "GND"
- board text added: "HI"
- board text added: "LO"
- board text added: "Mai 2026"
- board text added: "RST"
- board text added: "VBAT"
- board text added: "btaudio"
